File: Board Designs/Rear ECU/Rear ECU rev6.sch (EAGLE design)
At the start: 97 parts, among them X1 CONNECTOR-2, X2 CONNECTOR-6, X3 CONNECTOR-10MX150L_VERTICAL-10, X4 CONNECTOR-10MX150L_VERTICAL-10

Commit message: jparkerjones: Began updates on Front ECU, Moved Software Latch to Rear ECU
Parts:
- removed FSAE_FUSE: 8A, HyTechDevices:FUSE_MINIBLADE
- removed X2: CONNECTOR-6, HyTechDevices:CONNECTOR-6
- added D10: DIODE0805, HyTechDevices:DIODE0805
- added LED17, LED18: RED, HyTechDevices:LED-0805
- added R25: 330, HyTechDevices:RESISTOR0805-RES
- added R26, R31: 1.2K, HyTechDevices:RESISTOR0805-RES
- added SOFTWARE_SHUTOFF: G5LE, HyTechDevices:G5LE
- added U$5: CPC1002N, HyTechDevices:CPC1002N
Connections:
- new net N$40: LED18.A, R31.2
- new net N$43: D10.C, R26.1, SOFTWARE_SHUTOFF.COIL-, U$5.DC-
- new net N$44: R25.2, U$5.CONTROL-
- new net N$46: LED17.A, R26.2
- new net SHUTDOWN_D: R31.1, SOFTWARE_SHUTOFF.S, X3-3.S
- new net SOFTWARE_SHUTDOWN: U$3.A7, U$5.CONTROL+
- net +12V: now also U$5.DC+; no longer FSAE_FUSE.P1
- net 12VSUPPLY_FSAE: no longer FSAE_FUSE.P2
- net BMS_OK: no longer X2-2.S
- net BRAKE_LIGHT: no longer X2-4.S
- net GND: now also D10.A, LED17.C, LED18.C, R25.1, SOFTWARE_SHUTOFF.COIL+
- net GPIO_1: no longer X2-6.S
- net INVERTER_SUPPLY: no longer X2-5.S
- net OKHS: no longer X2-1.S
- net SHUTDOWN_C: now also SOFTWARE_SHUTOFF.P; no longer X2-3.S, X3-3.S
Other:
- note removed: "Install FSAE_FUSE for FSAE"

Commit message: Beginning work on Rear ECU
Parts:
- removed X4: CONNECTOR-10MX150L_VERTICAL-10, HyTechDevices:CONNECTOR-10MX150L_VERTICAL-10
- X1: value CONNECTOR-2 -> CONNECTOR-8MX150L_RIGHT_ANGLE-8; device HyTechDevices:CONNECTOR-2 -> HyTechDevices:CONNECTOR-8MX150L_RIGHT_ANGLE-8
- X3: value CONNECTOR-10MX150L_VERTICAL-10 -> CONNECTOR-10MX150L-RIGHT_ANGLE-10; device HyTechDevices:CONNECTOR-10MX150L_VERTICAL-10 -> HyTechDevices:CONNECTOR-10MX150L-RIGHT_ANGLE-10
Connections:
- removed net 12VSUPPLY_FSAE: X4-1.S
- net 12VSUPPLY_BRB: now also X1-7.S; no longer X1-1.S, X4-2.S
- net 12V_F1: now also X1-3.S; no longer X4-5.S
- net 12V_F2: now also X1-2.S; no longer X4-4.S
- net CANH: now also X1-6.S; no longer X4-8.S
- net CANL: now also X1-5.S; no longer X4-7.S
- net GND: now also X1-1.S, X1-4.S; no longer X1-2.S, X4-3.S, X4-6.S
- net GPIO_2: no longer X4-9.S
- net LATCH_EXT_BUTTON: now also X1-8.S; no longer X4-10.S
Other:
- moved on the sheet: X1-1, X1-2
Changed lines of the file:
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@@
 <part name="P+14" library="supply1" deviceset="+12V" device=""/>
 <part name="P+5" library="supply1" deviceset="+12V" device=""/>
-<part name="X1" library="HyTechDevices" deviceset="CONNECTOR-2" device=""/>
-<part name="GND25" library="HyTechSymbols" deviceset="GND" device=""/>
 <part name="D4" library="HyTechDevices" deviceset="DIODE" device="0805"/>
 <part name="D5" library="HyTechDevices" deviceset="DIODE" device="0805"/>
@@
 <part name="U$6" library="HyTechDevices" deviceset="G5LE" device=""/>
 <part name="U$7" library="HyTechDevices" deviceset="G5LE" device=""/>
-<part name="X3" library="HyTechDevices" deviceset="CONNECTOR-10" device="MX150L_VERTICAL-10"/>
-<part name="X4" library="HyTechDevices" deviceset="CONNECTOR-10" device="MX150L_VERTICAL-10"/>
+<part name="X3" library="HyTechDevices" deviceset="CONNECTOR-10" device="MX150L-RIGHT_ANGLE-10" value="CONNECTOR-10MX150L-RIGHT_ANGLE-10"/>
 <part name="GND32" library="HyTechSymbols" deviceset="GND" device=""/>
 <part name="GND33" library="HyTechSymbols" deviceset="GND" device=""/>
@@
 <part name="GND45" library="HyTechSymbols" deviceset="GND" device=""/>
 <part name="R31" library="HyTechDevices" deviceset="RESISTOR" device="0805-RES" value="1.2K"/>
+<part name="X1" library="HyTechDevices" deviceset="CONNECTOR-8" device="MX150L_RIGHT_ANGLE-8"/>
 </parts>
 <sheets>
@@
 <instance part="P+14" gate="1" x="137.16" y="200.66" rot="R180"/>
 <instance part="P+5" gate="1" x="355.6" y="104.14" rot="R90"/>
-<instance part="X1" gate="-2" x="48.26" y="78.74" rot="MR0"/>
-<instance part="X1" gate="-1" x="48.26" y="81.28" rot="MR0"/>
-<instance part="GND25" gate="1" x="53.34" y="76.2"/>
 <instance part="D4" gate="1" x="134.62" y="137.16"/>
 <instance part="D5" gate="1" x="393.7" y="60.96"/>
@@
 <instance part="X3" gate="-9" x="48.26" y="48.26" rot="MR0"/>
 <instance part="X3" gate="-10" x="48.26" y="45.72" rot="MR0"/>
-<instance part="X4" gate="-1" x="48.26" y="154.94" rot="MR0"/>
-<instance part="X4" gate="-2" x="48.26" y="152.4" rot="MR0"/>
-<instance part="X4" gate="-3" x="48.26" y="149.86" rot="MR0"/>
-<instance part="X4" gate="-4" x="48.26" y="147.32" rot="MR0"/>
-<instance part="X4" gate="-5" x="48.26" y="144.78" rot="MR0"/>
-<instance part="X4" gate="-6" x="48.26" y="142.24" rot="MR0"/>
-<instance part="X4" gate="-7" x="48.26" y="139.7" rot="MR0"/>
-<instance part="X4" gate="-8" x="48.26" y="137.16" rot="MR0"/>
-<instance part="X4" gate="-9" x="48.26" y="134.62" rot="MR0"/>
-<instance part="X4" gate="-10" x="48.26" y="132.08" rot="MR0"/>
 <instance part="GND32" gate="1" x="71.12" y="149.86" rot="R90"/>
 <instance part="GND33" gate="1" x="71.12" y="142.24" rot="R90"/>
@@
 <instance part="GND45" gate="1" x="495.3" y="45.72" rot="MR270"/>
 <instance part="R31" gate="G$1" x="474.98" y="45.72" rot="MR180"/>
+<instance part="X1" gate="-1" x="48.26" y="149.86" rot="MR0"/>
+<instance part="X1" gate="-2" x="48.26" y="147.32" rot="MR0"/>
+<instance part="X1" gate="-3" x="48.26" y="144.78" rot="MR0"/>
+<instance part="X1" gate="-4" x="48.26" y="142.24" rot="MR0"/>
+<instance part="X1" gate="-5" x="48.26" y="139.7" rot="MR0"/>
+<instance part="X1" gate="-6" x="48.26" y="137.16" rot="MR0"/>
+<instance part="X1" gate="-7" x="48.26" y="134.62" rot="MR0"/>
+<instance part="X1" gate="-8" x="48.26" y="132.08" rot="MR0"/>
 </instances>
 <busses>
@@
 </segment>
 <segment>
-<pinref part="X1" gate="-2" pin="S"/>
-<pinref part="GND25" gate="1" pin="GND"/>
-<wire x1="53.34" y1="78.74" x2="50.8" y2="78.74" width="0.1524" layer="91"/>
-</segment>
-<segment>
 <pinref part="XB" gate="G$1" pin="GND"/>
 <pinref part="GND11" gate="1" pin="GND"/>
@@
 </segment>
 <segment>
-<pinref part="X4" gate="-3" pin="S"/>
 <pinref part="GND32" gate="1" pin="GND"/>
 <wire x1="68.58" y1="149.86" x2="50.8" y2="149.86" width="0.1524" layer="91"/>
-</segment>
-<segment>
-<pinref part="X4" gate="-6" pin="S"/>
+<pinref part="X1" gate="-1" pin="S"/>
+</segment>
+<segment>
 <pinref part="GND33" gate="1" pin="GND"/>
 <wire x1="68.58" y1="142.24" x2="50.8" y2="142.24" width="0.1524" layer="91"/>
+<pinref part="X1" gate="-4" pin="S"/>
 </segment>
 <segment>
@@
 </segment>
 <segment>
-<pinref part="X4" gate="-7" pin="S"/>
 <wire x1="50.8" y1="139.7" x2="53.34" y2="139.7" width="0.1524" layer="91"/>
 <label x="53.34" y="139.7" size="1.27" layer="95" xref="yes"/>
+<pinref part="X1" gate="-5" pin="S"/>
 </segment>
 <segment>
@@
 <net name="CANH" class="0">
 <segment>
-<pinref part="X4" gate="-8" pin="S"/>
 <wire x1="50.8" y1="137.16" x2="53.34" y2="137.16" width="0.1524" layer="91"/>
 <label x="53.34" y="137.16" size="1.27" layer="95" xref="yes"/>
+<pinref part="X1" gate="-6" pin="S"/>
 </segment>
 <segment>
@@
 <net name="12V_F1" class="0">
 <segment>
-<pinref part="X4" gate="-5" pin="S"/>
 <wire x1="53.34" y1="144.78" x2="50.8" y2="144.78" width="0.1524" layer="91"/>
 <label x="53.34" y="144.78" size="1.27" layer="95" xref="yes"/>
+<pinref part="X1" gate="-3" pin="S"/>
 </segment>
 <segment>
@@
 <net name="12V_F2" class="0">
 <segment>
-<pinref part="X4" gate="-4" pin="S"/>
 <wire x1="53.34" y1="147.32" x2="50.8" y2="147.32" width="0.1524" layer="91"/>
 <label x="53.34" y="147.32" size="1.27" layer="95" xref="yes"/>
+<pinref part="X1" gate="-2" pin="S"/>
 </segment>
 <segment>
@@
 <net name="12VSUPPLY_BRB" class="0">
 <segment>
-<pinref part="X4" gate="-2" pin="S"/>
-<wire x1="53.34" y1="152.4" x2="50.8" y2="152.4" width="0.1524" layer="91"/>
-<label x="53.34" y="152.4" size="1.27" layer="95" xref="yes"/>
-</segment>
-<segment>
-<pinref part="X1" gate="-1" pin="S"/>
-<wire x1="50.8" y1="81.28" x2="53.34" y2="81.28" width="0.1524" layer="91"/>
-<label x="53.34" y="81.28" size="1.27" layer="95" xref="yes"/>
+<wire x1="53.34" y1="134.62" x2="50.8" y2="134.62" width="0.1524" layer="91"/>
+<label x="53.34" y="134.62" size="1.27" layer="95" xref="yes"/>
+<pinref part="X1" gate="-7" pin="S"/>
 </segment>
 <segment>
@@
 <net name="GPIO_2" class="0">
 <segment>
-<pinref part="X4" gate="-9" pin="S"/>
-<wire x1="50.8" y1="134.62" x2="53.34" y2="134.62" width="0.1524" layer="91"/>
-<label x="53.34" y="134.62" size="1.27" layer="95" xref="yes"/>
-</segment>
-<segment>
 <pinref part="U$11" gate="G$1" pin="P$2"/>
 <wire x1="246.38" y1="132.08" x2="254" y2="132.08" width="0.1524" layer="91"/>
@@
 </segment>
 <segment>
-<pinref part="X4" gate="-10" pin="S"/>
 <wire x1="50.8" y1="132.08" x2="53.34" y2="132.08" width="0.1524" layer="91"/>
 <label x="53.34" y="132.08" size="1.27" layer="95" xref="yes"/>
+<pinref part="X1" gate="-8" pin="S"/>
 </segment>
 <segment>
@@
 </segment>
 </net>
-<net name="12VSUPPLY_FSAE" class="0">
-<segment>
-<pinref part="X4" gate="-1" pin="S"/>
-<wire x1="53.34" y1="154.94" x2="50.8" y2="154.94" width="0.1524" layer="91"/>
-<label x="53.34" y="154.94" size="1.27" layer="95" xref="yes"/>
-</segment>
-</net>
