File: Board Designs/BMS/BMS Adapter for Enerdel/BMS Adapter.brd (EAGLE design)
At the start: 110 x 274.8 mm, 23 parts

Commit message: added Adapter file
Parts:
- added JP3, JP4: (no value), HyTechDevices:1X06
- added U$3, U$4: M07, HyTechDevices:1X07
Connections:
- removed net N$1: CELL0.P$1, U$1.1
- removed net N$10: CELL5.P$1, JP1.3
- removed net N$11: CELL7.P$1, JP1.4
- removed net N$12: CELL9.P$1, JP1.5
- removed net N$13: CELL11.P$1, JP1.6
- removed net N$14: CELL18.P$1, U$2.4
- removed net N$15: CELL16.P$1, U$2.3
- removed net N$16: CELL14.P$1, U$2.2
- removed net N$17: CELL13.P$1, JP2.1
- removed net N$18: CELL15.P$1, JP2.2
- removed net N$19: CELL17.P$1, JP2.3
- removed net N$2: CELL2.P$1, U$1.2
- removed net N$3: CELL4.P$1, U$1.3
- removed net N$4: CELL6.P$1, U$1.4
- removed net N$5: CELL8.P$1, U$1.5
- removed net N$6: CELL10.P$1, U$1.6
- removed net N$7: CELL12.P$1, U$1.7
- removed net N$8: CELL1.P$1, JP1.1
- removed net N$9: CELL3.P$1, JP1.2
- new net CELL0: CELL0.P$1, U$1.1, U$4.1
- new net CELL1: CELL1.P$1, JP1.1, JP4.1
- new net CELL10: CELL10.P$1, U$1.6, U$4.6
- new net CELL11: CELL11.P$1, JP1.6, JP4.6
- new net CELL12: CELL12.P$1, CELL13.P$1, JP2.1, JP3.1, U$1.7, U$4.7
- new net CELL14: CELL14.P$1, U$2.2, U$3.2
- new net CELL15: CELL15.P$1, JP2.2, JP3.2
- new net CELL16: CELL16.P$1, U$2.3, U$3.3
- new net CELL17: CELL17.P$1, JP2.3, JP3.3
- new net CELL18: CELL18.P$1, U$2.4, U$3.4
- new net CELL2: CELL2.P$1, U$1.2, U$4.2
- new net CELL3: CELL3.P$1, JP1.2, JP4.2
- new net CELL4: CELL4.P$1, U$1.3, U$4.3
- new net CELL5: CELL5.P$1, JP1.3, JP4.3
- new net CELL6: CELL6.P$1, U$1.4, U$4.4
- new net CELL7: CELL7.P$1, JP1.4, JP4.4
- new net CELL8: CELL8.P$1, U$1.5, U$4.5
- new net CELL9: CELL9.P$1, JP1.5, JP4.5
Routing:
- net CELL12: track 0.00 -> 491.5 mm, vias 0 -> 3
- net CELL11: track 0.00 -> 279.4 mm, vias 0 -> 2
- net CELL9: track 0.00 -> 255.0 mm, vias 0 -> 2
- net CELL10: track 0.00 -> 249.9 mm, vias 0 -> 2
- net CELL8: track 0.00 -> 231.5 mm, vias 0 -> 2
- net CELL7: track 0.00 -> 222.4 mm, vias 0 -> 2
- net N$7: track 215.9 -> 0.00 mm, vias 1 -> 0
- net N$13: track 211.4 -> 0.00 mm, vias 1 -> 0
- net CELL5: track 0.00 -> 203.3 mm, vias 0 -> 2
- net CELL6: track 0.00 -> 197.2 mm, vias 0 -> 2
- net CELL14: track 0.00 -> 189.6 mm, vias 0 -> 2
- net N$12: track 184.2 -> 0.00 mm, vias 1 -> 0
- net N$6: track 178.6 -> 0.00 mm, vias 1 -> 0
- net CELL3: track 0.00 -> 175.8 mm, vias 0 -> 2
- net CELL4: track 0.00 -> 171.1 mm, vias 0 -> 2
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
Commit message: Changed adapter board to include minifit connectors.
Parts:
- removed JP1, JP2, JP3, JP4: (no value), HyTechDevices:1X06
- removed U$1, U$2, U$3, U$4: M07, HyTechDevices:1X07
- added X1, X2, X3, X4: CONNECTOR-4, HyTechDevices:MINIFIT_5566-4
- added X5, X6: CONNECTOR-6, HyTechDevices:MINIFIT_5566-6
- added X7, X8: CONNECTOR-8, HyTechDevices:MINIFIT_5566-8
Connections:
- net CELL0: now also X7.8, X8.8; no longer U$1.1, U$4.1
- net CELL1: now also X5.6, X6.6; no longer JP1.1, JP4.1
- net CELL10: now also X7.3, X8.3; no longer U$1.6, U$4.6
- net CELL11: now also X5.1, X6.1; no longer JP1.6, JP4.6
- net CELL12: now also X1.4, X2.4, X7.2, X8.2; no longer JP2.1, JP3.1, U$1.7, U$4.7
- net CELL14: now also X3.4, X4.4; no longer U$2.2, U$3.2
- net CELL15: now also X1.3, X2.3; no longer JP2.2, JP3.2
- net CELL16: now also X3.3, X4.3; no longer U$2.3, U$3.3
- net CELL17: now also X1.2, X2.2; no longer JP2.3, JP3.3
- net CELL18: now also X3.2, X4.2; no longer U$2.4, U$3.4
- net CELL2: now also X7.7, X8.7; no longer U$1.2, U$4.2
- net CELL3: now also X5.5, X6.5; no longer JP1.2, JP4.2
- net CELL4: now also X7.6, X8.6; no longer U$1.3, U$4.3
- net CELL5: now also X5.4, X6.4; no longer JP1.3, JP4.3
- net CELL6: now also X7.5, X8.5; no longer U$1.4, U$4.4
- net CELL7: now also X5.3, X6.3; no longer JP1.4, JP4.4
- net CELL8: now also X7.4, X8.4; no longer U$1.5, U$4.5
- net CELL9: now also X5.2, X6.2; no longer JP1.5, JP4.5
Routing:
- net CELL8: track 231.5 -> 271.9 mm, vias 2 -> 3
- net CELL14: track 189.6 -> 152.0 mm, vias 2 -> 1
- net CELL18: track 107.3 -> 143.3 mm, vias 2 -> 1
- net CELL0: track 137.3 -> 108.3 mm
- net CELL1: track 143.4 -> 118.2 mm
- net CELL5: track 203.3 -> 180.9 mm
- net CELL2: track 145.0 -> 126.8 mm
- net CELL4: track 171.1 -> 153.2 mm
- net CELL6: track 197.2 -> 179.7 mm
- net CELL10: track 249.9 -> 265.8 mm
- net CELL9: track 255.0 -> 270.3 mm
- net CELL3: track 175.8 -> 161.5 mm
- net CELL12: track 491.5 -> 485.0 mm
- net CELL11: track 279.4 -> 285.6 mm, vias 2 -> 4
- net CELL17: track 86.9 -> 92.5 mm
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