File: Board Designs/BMS/BMS Adapter for Enerdel/BMS Adapter rev3.sch (EAGLE design)
At the start: 27 parts

Commit message: Add Molex 14-pin to library, add layout for battery testing board, update silkscreen on BMS adapter board
Other:
- note added: "Warning: only install Mode A or Mode B connectors Do not use connectors from both modes"
- note removed: "Warning: install only the 2 connectors for one mode"
Changed lines of the file:
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@@
 <text x="2.54" y="160.02" size="7.62" layer="90">A Mode</text>
 <text x="205.74" y="160.02" size="7.62" layer="90">B Mode</text>
-<text x="167.64" y="177.8" size="7.62" layer="90" align="center">Warning: install only the 2 connectors for one mode</text>
+<text x="167.64" y="187.96" size="7.62" layer="90" align="center">Warning: only install Mode A or Mode B connectors
+Do not use connectors from both modes</text>
 </plain>
 <instances>
@@
 </schematic>
 </drawing>
+<compatibility>
+<note version="6.3" minversion="6.2.2" severity="warning">
+Since Version 6.2.2 text objects can contain more than one line,
+which will not be processed correctly with this version.
+</note>
+</compatibility>
 </eagle>
