File: Board Designs/BMS/BMS Adapter for Enerdel/BMS Adapter rev3.brd (EAGLE design)
At the start: 110 x 320.5 mm, 27 parts

Commit message: Add 10k resistors to current sensors, fix DRC errors, small silkscreen tweaks for mfg
Other:
- board text added: "BMS Enerdel Adapter 2019 rev3"
- board text removed: "BMS Enerdel Adapter rev3"
