File: Board Designs/Main ECU/MainECU rev1.brd (EAGLE design)
At the start: 142.2 x 88.6 mm, 144 parts, among them X1 CONNECTOR-37, X2 CONNECTOR-4AUTOSPORT, X3 CONNECTOR-4NANO-FIT-VERTICAL-4, X4 CONNECTOR-4NANO-FIT-VERTICAL-4

Commit message: Update to Layout
Parts:
- BRAKE_LIGHT_SSR: value SOLID_STATE_RELAY_VO14642AT -> CPC1002N; device HyTechDevices:DIL06 -> HyTechDevices:SOP04
- REG: device HyTechDevices:SOT223 -> HyTechDevices:OKI-78SR
- U$17: value MCP23S17DIP -> MCP23S17SOIC_WIDE; device HyTechDevices:DIL28-3 -> HyTechDevices:SOIC-28W
- moved R33 280.6 mm to (113.3, 6.60), flipped to the bottom, turned to 180 degrees
- moved LED12 264.5 mm to (120.7, 25.3), turned to 180 degrees
- moved R27 259.8 mm to (120.7, 21.3), turned to 270 degrees
- moved R28 258.7 mm to (115.6, 21.3), turned to 270 degrees
- moved D7 253.0 mm to (112.0, 35.8), flipped to the bottom, turned to 270 degrees
- moved D9 251.5 mm to (111.5, 53.6), flipped to the bottom, turned to 270 degrees
- moved R1 249.2 mm to (100.3, 22.9), turned to 180 degrees
- moved R2 249.2 mm to (96.5, 22.9)
- moved R24 247.8 mm to (118.1, 21.3), turned to 270 degrees
- moved C7 243.1 mm to (96.8, 58.2), flipped to the bottom, turned to 270 degrees
- moved D8 241.7 mm to (111.5, 70.1), flipped to the bottom, turned to 270 degrees
- moved R3 237.4 mm to (99.8, 65.8), flipped to the bottom, turned to 180 degrees
- moved U$10 228.9 mm to (101.3, 59.7), flipped to the bottom, turned to 270 degrees
- moved U$6 228.2 mm to (104.4, 26.7)
- moved CAN_TRANSCEIVER 227.1 mm to (106.7, 23.1), flipped to the bottom, turned to 270 degrees
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Connections:
- removed net N$41: C13.2, C5.1, REG1.3, REG2.3
- removed net N$92: X1.P$6
- removed net N$94: X1.P$4
- removed net N$95: X1.P$3
- removed net N$96: X1.P$2
- removed net PEDALS_GND: X1.P$15, X1.P$16, X1.P$17
- new net TELEMETRY5V: ADXL345_BREAKOUT.1, C10.1, C13.2, C5.1, C9.1, CAN_TRANSCEIVER.3, REG1.3, REG2.3, U$10.8, U$2.VIN, U$9.8
- net +12V: now also BRAKE_LIGHT_SSR.4, X1.P$9; no longer BRAKE_LIGHT_SSR.6, X1.P$5
- net +5V: now also U$1.VIN, X1.P$15; no longer ADXL345_BREAKOUT.1, C10.1, C9.1, CAN_TRANSCEIVER.3, U$10.8, U$9.8, X1.P$12
- net BRAKE_LIGHT: now also BRAKE_LIGHT_SSR.3, X1.P$2; no longer BRAKE_LIGHT_SSR.5
- net CANH: now also X1.P$12, X1.P$26; no longer X1.P$8
- net CANL: now also X1.P$11, X1.P$25; no longer X1.P$7
- net COOLINGSENSE: now also U$2.A12; no longer U$2.A2
- net DASH_CTRL10: now also X1.P$29; no longer X1.P$30
- net DASH_CTRL11: now also X1.P$36; no longer X1.P$31
- net DASH_CTRL12: now also X1.P$35; no longer X1.P$32
- net DASH_CTRL9: now also X1.P$30; no longer X1.P$29
- net DASH_IO1: now also X1.P$23; no longer X1.P$21
- net DASH_IO2: now also X1.P$24; no longer X1.P$22
- net DASH_IO3: now also X1.P$22; no longer X1.P$23
- net DASH_IO4: now also X1.P$21; no longer X1.P$24
- net DASH_IO5: now also X1.P$33; no longer X1.P$25
- net DASH_IO6: now also X1.P$34; no longer X1.P$26
- net ECUSENSE: now also U$2.A13; no longer U$2.A1
- net FAN1-: now also 5AFUSE.R1, 5AFUSE.R2; no longer X2.P$2
- net GND: now also U$17.15, U$17.16, U$17.17, X1.P$16, X1.P$17, X1.P$18, X1.P$19, X1.P$31; no longer REG.4
- net INVERTER_SUPPLY: now also X1.P$4; no longer X1.P$1
- net LATCH_EXT_BUTTON: now also X1.P$5; no longer X1.P$18
- net N$1: now also X1.P$1
- net OKHS: now also X1.P$10; no longer X1.P$19
- net PUMP1-: now also X2.P$2; no longer 5AFUSE.R1, 5AFUSE.R2
- net READ_ACCEL1: now also X1.P$7; no longer X1.P$10
- net READ_ACCEL2: now also X1.P$6; no longer X1.P$9
- net READ_BRAKE: now also X1.P$8; no longer X1.P$11
- net SHUTDOWN_D: now also X1.P$3
Routing:
- net GND: track 0.00 -> 452.1 mm, vias 0 -> 3
- net +12V: track 0.00 -> 230.4 mm, vias 0 -> 4
- net RELAY_CTRL3: track 0.00 -> 167.8 mm, vias 0 -> 2
- net RELAY_CTRL2: track 0.00 -> 165.7 mm, vias 0 -> 2
- net TELEMETRY5V: track 0.00 -> 164.0 mm, vias 0 -> 3
- net RELAY_CTRL1: track 0.00 -> 155.9 mm, vias 0 -> 2
- net +5V: track 0.00 -> 131.6 mm, vias 0 -> 1
- net CANL: track 0.00 -> 130.4 mm, vias 0 -> 1
- net CANH: track 0.00 -> 129.5 mm, vias 0 -> 1
- net SCL: track 0.00 -> 108.5 mm
- net SDA: track 0.00 -> 108.3 mm, vias 0 -> 1
- net COOLINGSENSE: track 0.00 -> 102.7 mm, vias 0 -> 1
- net BRAKE_LIGHT_CTRL: track 0.00 -> 82.4 mm
- net INVERTER_SUPPLY: track 0.00 -> 76.4 mm
- net SHUTDOWN_D: track 0.00 -> 73.8 mm
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Other:
- board size 142.2 x 88.6 mm -> 120.6 x 78.9 mm

Commit message: Completed Main ECU Layout
Parts:
- U$17: value MCP23S17SOIC_WIDE -> MCP23S17SSOP28; device HyTechDevices:SOIC-28W -> HyTechDevices:SSOP28
- moved R32 198.9 mm to (34.3, 30.5), turned to 270 degrees
- moved C1 196.4 mm to (71.1, 23.4)
- moved C12 196.2 mm to (74.4, 68.3), flipped to the bottom
- moved C2 192.1 mm to (66.0, 28.7), turned to 270 degrees
- moved R20 190.6 mm to (69.1, 30.2)
- moved R30 189.9 mm to (30.2, 30.5), turned to 270 degrees
- moved U$19 188.8 mm to (68.1, 38.9), turned to 180 degrees
- moved ACC2_PU 184.6 mm to (88.1, 58.4)
- moved LED10 182.6 mm to (34.3, 26.4)
- moved C4 180.5 mm to (70.6, 70.4), flipped to the bottom, turned to 180 degrees
- moved ACC2_PD 180.5 mm to (86.1, 56.4), turned to 180 degrees
- moved U$14 177.5 mm to (66.8, 37.1), turned to 180 degrees
- moved U$13 175.9 mm to (66.8, 35.3), turned to 180 degrees
- moved ACC1_PU 175.2 mm to (88.4, 64.5)
- moved C3 174.9 mm to (70.6, 75.7), flipped to the bottom, turned to 180 degrees
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Connections:
- removed net SOFTWARESHUTDOWN: U$1.A7
- net BRAKE_LIGHT: now also X1.P$8; no longer X1.P$2
- net GND: now also U$23.4
- net READ_ACCEL1: now also U$18.2; no longer U$18.1, X1.P$7
- net READ_ACCEL2: now also U$18.3; no longer U$18.2, X1.P$6
- net READ_BRAKE: now also U$18.1; no longer U$18.3, X1.P$8
- net SIGNAL_ACCEL1: now also X1.P$7
- net SIGNAL_ACCEL2: now also X1.P$6
- net SIGNAL_BRAKE: now also X1.P$2
- net SOFTWARE_SHUTDOWN: now also U$1.A7
Routing:
- net GND: track 452.1 -> 724.6 mm, vias 3 -> 9
- net +12V: track 230.4 -> 431.4 mm, vias 4 -> 12
- net +5V: track 131.6 -> 296.5 mm, vias 1 -> 7
- net TEMPSENSE: track 0.00 -> 109.9 mm, vias 0 -> 2
- net BMS_OK: track 39.4 -> 100.4 mm, vias 1 -> 2
- net LATCH_EXT_BUTTON: track 17.2 -> 73.6 mm
- net SOFTWARE_SHUTDOWN: track 0.00 -> 51.0 mm, vias 0 -> 1
- net INVERTER_CTRL: track 0.00 -> 45.4 mm
- net N$23: track 0.00 -> 41.1 mm
- net N$24: track 0.00 -> 39.6 mm
- net N$47: track 0.00 -> 39.2 mm, vias 0 -> 1
- net N$16: track 0.00 -> 32.2 mm, vias 0 -> 1
- net DASH_IO5: track 0.00 -> 31.1 mm, vias 0 -> 2
- net SIGNAL_ACCEL2: track 0.00 -> 25.3 mm, vias 0 -> 1
- net N$9: track 0.00 -> 24.6 mm, vias 0 -> 1
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
Commit message: Updated Rev 2 Schematic/Rev 1 Layout
Parts:
- moved C8 7.75 mm to (93.0, 36.8)
- moved X2 7.68 mm to (98.6, 41.9), turned to 225 degrees
- moved U$9 7.62 mm to (92.7, 33.3)
- moved R9 7.15 mm to (93.2, 63.0)
- moved C9 6.62 mm to (98.6, 31.8)
- moved BOARD_TEMP 6.48 mm to (94.0, 65.3)
- moved C7 5.40 mm to (93.2, 61.7)
- moved R4 4.50 mm to (99.6, 67.1)
- moved R3 4.26 mm to (95.8, 67.1)
- moved U$10 4.13 mm to (98.6, 62.7)
- moved S1 3.39 mm to (32.0, 38.1)
- moved ADXL345_BREAKOUT 2.30 mm to (52.1, 29.0), turned to 0 degrees
- moved C10 2.27 mm to (93.7, 58.2), turned to 180 degrees
- moved LED11 1.52 mm to (28.7, 26.4)
- moved R30 1.52 mm to (28.7, 30.5)
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Connections:
- removed net DFASH_IO8: X1.P$28
- net +12V: now also X1.P$7; no longer X1.P$9
- net +5V: now also X1.P$11, X1.P$12; no longer X1.P$14, X1.P$15
- net BMS_OK: now also X1.P$19; no longer X1.P$20
- net BRAKE_LIGHT: now also X1.P$6; no longer X1.P$8
- net CANH: now also X1.P$10, X1.P$25; no longer X1.P$12, X1.P$26
- net CANL: now also X1.P$24, X1.P$9; no longer X1.P$11, X1.P$25
- net DASH_CTRL10: now also X1.P$28; no longer X1.P$29
- net DASH_CTRL11: now also X1.P$35; no longer X1.P$36
- net DASH_CTRL12: now also X1.P$34; no longer X1.P$35
- net DASH_CTRL9: now also X1.P$29; no longer X1.P$30
- net DASH_IO1: now also X1.P$22; no longer X1.P$23
- net DASH_IO2: now also X1.P$23; no longer X1.P$24
- net DASH_IO3: now also X1.P$21; no longer X1.P$22
- net DASH_IO4: now also X1.P$20; no longer X1.P$21
- net DASH_IO5: now also X1.P$32; no longer X1.P$33
- net DASH_IO6: now also X1.P$33; no longer X1.P$34
- net DASH_IO7: now also X1.P$26; no longer X1.P$27
- net DASH_IO8: now also X1.P$27
- net GND: now also X1.P$14, X1.P$15, X1.P$30, X1.P$36; no longer X1.P$17, X1.P$18, X1.P$19, X1.P$31
- net INVERTER_SUPPLY: now also X1.P$2; no longer X1.P$4
- net LATCH_EXT_BUTTON: now also X1.P$3; no longer X1.P$5
- net N$1: now also X1.P$17; no longer X1.P$1
- net OKHS: now also X1.P$8; no longer X1.P$10
- net SHUTDOWN_D: now also X1.P$1; no longer X1.P$3
- net SIGNAL_ACCEL1: now also X1.P$5; no longer X1.P$7
- net SIGNAL_ACCEL2: now also X1.P$4; no longer X1.P$6
- net SIGNAL_BRAKE: now also X1.P$18; no longer X1.P$2
Routing:
- net SCL: track 112.8 -> 130.5 mm
- net SDA: track 114.2 -> 130.8 mm
- net DASH_IO8: track 24.4 -> 37.5 mm, vias 0 -> 2
- net 12VIN: track 23.4 -> 11.3 mm
- net N$3: track 7.42 -> 19.4 mm, vias 0 -> 2
- net PUMP1-: track 16.7 -> 8.14 mm
- net GND: track 724.6 -> 730.3 mm, vias 9 -> 11
- net CURRENTSENSE2: track 60.9 -> 66.3 mm
- net DASH_IO5: track 31.1 -> 35.4 mm
- net TELEMETRY5V: track 163.6 -> 167.8 mm, vias 3 -> 4
- net +5V: track 296.5 -> 292.7 mm
- net LATCH_EXT_BUTTON: track 73.6 -> 76.7 mm
- net TEMPSENSE: track 109.9 -> 107.1 mm
- net CANL: track 129.9 -> 127.2 mm
- net DASH_CTRL9: track 30.5 -> 33.1 mm, vias 0 -> 1
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Other:
- board text added: "Assoc"
- board text added: "BMS OK"
- board text added: "BMSCoil"
- board text added: "Designed By Parker Jones"
- board text added: "Fan1"
- board text added: "Fan2"
- board text added: "HyTech 2019 Main ECU rev1"
- board text added: "IMD Coil"
- board text added: "IMDOK"
- board text added: "Inverter"
- board text added: "Latch Button"
- board text added: "MQTT"
- board text added: "PUMP"
- board text added: "Shutdown"
- board text added: "Software"
