File: Board Designs/Main ECU/MainECU rev4.sch (EAGLE design)
At the start: 164 parts, among them Q10 MMBT3904LT3G, Q11 MMBT3904LT3G, Q9 MMBT3904LT3G, X1 CONNECTOR-37, X2 CONNECTOR-4AUTOSPORT, X3 CONNECTOR-4NANO-FIT-VERTICAL-4, X4 CONNECTOR-4NANO-FIT-VERTICAL-4

Commit message: Main ECU rev{1-5}: Update values of LED resistors based on testing
Parts:
- R11: value 43 -> 150
- R14, R21: value 820 -> 2k
- R16, R25, R32, R51, R52: value 100 -> 1.2k
- R17: value 820 -> 20k
- R31: value 1.2K -> 6.8k
- R45: value 33 -> 0
Changed lines of the file:
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@@
 <part name="BMS_SSR" library="HyTechDevices" deviceset="CPC1002N" device=""/>
 <part name="GND3" library="HyTechSymbols" deviceset="GND" device=""/>
-<part name="R11" library="HyTechDevices" deviceset="RESISTOR" device="0805-RES" value="43"/>
+<part name="R11" library="HyTechDevices" deviceset="RESISTOR" device="0805-RES" value="150"/>
 <part name="R12" library="HyTechDevices" deviceset="RESISTOR" device="0805-RES" value="33"/>
 <part name="BMS_LATCH_SSR" library="HyTechDevices" deviceset="CPC1002N" device=""/>
@@
 <part name="LED3" library="HyTechDevices" deviceset="LED" device="-0805" value="Green"/>
 <part name="LED5" library="HyTechDevices" deviceset="LED" device="-0805" value="Yellow"/>
-<part name="R14" library="HyTechDevices" deviceset="RESISTOR" device="0805-RES" value="820"/>
+<part name="R14" library="HyTechDevices" deviceset="RESISTOR" device="0805-RES" value="2k"/>
 <part name="GND6" library="HyTechSymbols" deviceset="GND" device=""/>
 <part name="IMD_SHUTDOWN1" library="HyTechDevices" deviceset="G2RL-2-DC12" device=""/>
 <part name="GND19" library="HyTechSymbols" deviceset="GND" device=""/>
-<part name="R17" library="HyTechDevices" deviceset="RESISTOR" device="0805-RES" value="820"/>
+<part name="R17" library="HyTechDevices" deviceset="RESISTOR" device="0805-RES" value="20k"/>
 <part name="LED7" library="HyTechDevices" deviceset="LED" device="-0805" value="Green"/>
 <part name="GND20" library="HyTechSymbols" deviceset="GND" device=""/>
@@
 <part name="LED9" library="HyTechDevices" deviceset="LED" device="-0805" value="Yellow"/>
 <part name="GND24" library="HyTechSymbols" deviceset="GND" device=""/>
-<part name="R21" library="HyTechDevices" deviceset="RESISTOR" device="0805-RES" value="820"/>
+<part name="R21" library="HyTechDevices" deviceset="RESISTOR" device="0805-RES" value="2k"/>
 <part name="P+10" library="supply1" deviceset="+12V" device=""/>
 <part name="P+5" library="supply1" deviceset="+12V" device=""/>
@@
 <part name="LED18" library="HyTechDevices" deviceset="LED" device="-0805" value="RED"/>
 <part name="GND45" library="HyTechSymbols" deviceset="GND" device=""/>
-<part name="R31" library="HyTechDevices" deviceset="RESISTOR" device="0805-RES" value="1.2K"/>
+<part name="R31" library="HyTechDevices" deviceset="RESISTOR" device="0805-RES" value="6.8k"/>
 <part name="GND1" library="HyTechSymbols" deviceset="GND" device=""/>
 <part name="GND4" library="HyTechSymbols" deviceset="GND" device=""/>
@@
 <part name="GND53" library="HyTechSymbols" deviceset="GND" device=""/>
 <part name="LED10" library="HyTechDevices" deviceset="LED" device="-0805" value="Red"/>
-<part name="R32" library="HyTechDevices" deviceset="RESISTOR" device="0805-RES" value="100"/>
+<part name="R32" library="HyTechDevices" deviceset="RESISTOR" device="0805-RES" value="1.2k"/>
 <part name="GND54" library="HyTechSymbols" deviceset="GND" device=""/>
 <part name="R33" library="HyTechDevices" deviceset="RESISTOR" device="0805-RES" value="4.7k"/>
@@
 <part name="P+35" library="supply1" library_urn="urn:adsk.eagle:library:371" deviceset="+5V" device=""/>
 <part name="LED14" library="HyTechDevices" deviceset="LED" device="-0805" value="Blue"/>
-<part name="R45" library="HyTechDevices" deviceset="RESISTOR" device="0805-RES" value="33"/>
+<part name="R45" library="HyTechDevices" deviceset="RESISTOR" device="0805-RES" value="0"/>
 <part name="GND62" library="HyTechSymbols" deviceset="GND" device=""/>
 <part name="X3" library="HyTechDevices" deviceset="CONNECTOR-4" device="NANO-FIT-VERTICAL-4"/>
@@
 <part name="LED6" library="HyTechDevices" deviceset="LED" device="-0805" value="Red"/>
 <part name="GND17" library="HyTechSymbols" deviceset="GND" device=""/>
-<part name="R16" library="HyTechDevices" deviceset="RESISTOR" device="0805-RES" value="100"/>
+<part name="R16" library="HyTechDevices" deviceset="RESISTOR" device="0805-RES" value="1.2k"/>
 <part name="P+8" library="supply1" deviceset="+12V" device=""/>
 <part name="P+12" library="supply1" deviceset="+12V" device=""/>
@@
 <part name="P+36" library="supply1" deviceset="+12V" device=""/>
 <part name="LED4" library="HyTechDevices" deviceset="LED" device="-0805" value="Red"/>
-<part name="R25" library="HyTechDevices" deviceset="RESISTOR" device="0805-RES" value="100"/>
+<part name="R25" library="HyTechDevices" deviceset="RESISTOR" device="0805-RES" value="1.2k"/>
 <part name="GND77" library="HyTechSymbols" deviceset="GND" device=""/>
 <part name="LED12" library="HyTechDevices" deviceset="LED" device="-0805" value="Red"/>
-<part name="R51" library="HyTechDevices" deviceset="RESISTOR" device="0805-RES" value="100"/>
+<part name="R51" library="HyTechDevices" deviceset="RESISTOR" device="0805-RES" value="1.2k"/>
 <part name="GND78" library="HyTechSymbols" deviceset="GND" device=""/>
 <part name="LED13" library="HyTechDevices" deviceset="LED" device="-0805" value="Red"/>
-<part name="R52" library="HyTechDevices" deviceset="RESISTOR" device="0805-RES" value="100"/>
+<part name="R52" library="HyTechDevices" deviceset="RESISTOR" device="0805-RES" value="1.2k"/>
 <part name="GND79" library="HyTechSymbols" deviceset="GND" device=""/>
 </parts>
