File: Board Designs/Main ECU/MainECU rev2.brd (EAGLE design)
At the start: 120.6 x 78.9 mm, 148 parts, among them X1 CONNECTOR-37, X2 CONNECTOR-4AUTOSPORT, X3 CONNECTOR-4NANO-FIT-VERTICAL-4, X4 CONNECTOR-4NANO-FIT-VERTICAL-4

Commit message: Add transistor P/Ns to main ECU rev2 schematic
Parts:
- Q1, Q2, Q3, Q4, Q5, Q6, Q7, Q8: value (none) -> MMBT3904LT3G
- U$4, U$6, U$7: value N-CHANNEL_MOSFET_HOR_HOLE -> N-CHANNEL_MOSFET_FQP30N06L
Changed lines of the file:
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@@
 <element name="X3" library="HyTechDevices" package="NANO-FIT_VERTICAL-4" value="CONNECTOR-4NANO-FIT-VERTICAL-4" x="78.486" y="48.514" smashed="yes" rot="R90"/>
 <element name="X4" library="HyTechDevices" package="NANO-FIT_VERTICAL-4" value="CONNECTOR-4NANO-FIT-VERTICAL-4" x="78.486" y="41.91" smashed="yes" rot="R90"/>
-<element name="U$4" library="HyTechDevices" package="TO-220-H-HOLE" value="N-CHANNEL_MOSFET_HOR_HOLE" x="105.918" y="55.626" smashed="yes" rot="MR90"/>
-<element name="U$7" library="HyTechDevices" package="TO-220-H-HOLE" value="N-CHANNEL_MOSFET_HOR_HOLE" x="105.918" y="71.628" smashed="yes" rot="MR90"/>
-<element name="U$6" library="HyTechDevices" package="TO-220-H-HOLE" value="N-CHANNEL_MOSFET_HOR_HOLE" x="105.918" y="41.656" smashed="yes" rot="MR90"/>
+<element name="U$4" library="HyTechDevices" package="TO-220-H-HOLE" value="N-CHANNEL_MOSFET_FQP30N06L" x="105.918" y="55.626" smashed="yes" rot="MR90"/>
+<element name="U$7" library="HyTechDevices" package="TO-220-H-HOLE" value="N-CHANNEL_MOSFET_FQP30N06L" x="105.918" y="71.628" smashed="yes" rot="MR90"/>
+<element name="U$6" library="HyTechDevices" package="TO-220-H-HOLE" value="N-CHANNEL_MOSFET_FQP30N06L" x="105.918" y="41.656" smashed="yes" rot="MR90"/>
 <element name="R24" library="HyTechDevices" package="0805" value="10k" x="87.122" y="67.564" smashed="yes" rot="R180">
 <attribute name="NAME" x="87.122" y="66.8401" size="0.3048" layer="25" rot="R180" align="bottom-center"/>
@@
 <attribute name="VALUE" x="75.6412" y="75.946" size="0.3048" layer="27" rot="R90" align="top-center"/>
 </element>
-<element name="Q1" library="HyTechDevices" package="SOT23" value="" x="78.74" y="76.2" smashed="yes" rot="MR180"/>
-<element name="Q2" library="HyTechDevices" package="SOT23" value="" x="73.914" y="70.612" smashed="yes" rot="MR90"/>
-<element name="Q3" library="HyTechDevices" package="SOT23" value="" x="65.278" y="70.104" smashed="yes" rot="MR180"/>
-<element name="Q4" library="HyTechDevices" package="SOT23" value="" x="62.484" y="69.088" smashed="yes" rot="MR180"/>
-<element name="Q5" library="HyTechDevices" package="SOT23" value="" x="78.486" y="75.692" smashed="yes" rot="R180"/>
+<element name="Q1" library="HyTechDevices" package="SOT23" value="MMBT3904LT3G" x="78.74" y="76.2" smashed="yes" rot="MR180"/>
+<element name="Q2" library="HyTechDevices" package="SOT23" value="MMBT3904LT3G" x="73.914" y="70.612" smashed="yes" rot="MR90"/>
+<element name="Q3" library="HyTechDevices" package="SOT23" value="MMBT3904LT3G" x="65.278" y="70.104" smashed="yes" rot="MR180"/>
+<element name="Q4" library="HyTechDevices" package="SOT23" value="MMBT3904LT3G" x="62.484" y="69.088" smashed="yes" rot="MR180"/>
+<element name="Q5" library="HyTechDevices" package="SOT23" value="MMBT3904LT3G" x="78.486" y="75.692" smashed="yes" rot="R180"/>
 <element name="R41" library="HyTechDevices" package="0805" value="2.2k" x="69.85" y="69.85" smashed="yes">
 <attribute name="NAME" x="69.85" y="70.5739" size="0.3048" layer="25" align="bottom-center"/>
 <attribute name="VALUE" x="69.85" y="69.1388" size="0.3048" layer="27" align="top-center"/>
 </element>
-<element name="Q6" library="HyTechDevices" package="SOT23" value="" x="74.93" y="70.358" smashed="yes" rot="R270"/>
+<element name="Q6" library="HyTechDevices" package="SOT23" value="MMBT3904LT3G" x="74.93" y="70.358" smashed="yes" rot="R270"/>
 <element name="R42" library="HyTechDevices" package="0805" value="2.2k" x="62.23" y="71.12" smashed="yes">
 <attribute name="NAME" x="62.23" y="71.8439" size="0.3048" layer="25" align="bottom-center"/>
 <attribute name="VALUE" x="62.23" y="70.4088" size="0.3048" layer="27" align="top-center"/>
 </element>
-<element name="Q7" library="HyTechDevices" package="SOT23" value="" x="65.532" y="68.072" smashed="yes" rot="R180"/>
+<element name="Q7" library="HyTechDevices" package="SOT23" value="MMBT3904LT3G" x="65.532" y="68.072" smashed="yes" rot="R180"/>
 <element name="R44" library="HyTechDevices" package="0805" value="2.2k" x="57.15" y="66.548" smashed="yes" rot="R270">
 <attribute name="NAME" x="57.8739" y="66.548" size="0.3048" layer="25" rot="R270" align="bottom-center"/>
 <attribute name="VALUE" x="56.4388" y="66.548" size="0.3048" layer="27" rot="R270" align="top-center"/>
 </element>
-<element name="Q8" library="HyTechDevices" package="SOT23" value="" x="61.468" y="65.532" smashed="yes" rot="R270"/>
+<element name="Q8" library="HyTechDevices" package="SOT23" value="MMBT3904LT3G" x="61.468" y="65.532" smashed="yes" rot="R270"/>
 <element name="U$11" library="HyTechDevices" package="0805" value="JUMPER" x="70.612" y="67.818" smashed="yes" rot="R180">
 <attribute name="NAME" x="70.612" y="67.0941" size="0.3048" layer="25" rot="R180" align="bottom-center"/>

Commit message: Main ECU: [rev2, rev3] Fix filter frequency capacitor values, [rev1b, rev3] shorten a few traces
Parts:
- C14, C17, C3: value 5.3uF -> 47pF
Changed lines of the file:
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@@
 <attribute name="VALUE" x="64.008" y="40.386" size="0.6096" layer="28" rot="MR90" align="bottom-center"/>
 </element>
-<element name="C3" library="HyTechDevices" package="0805" value="5.3uF" x="55.372" y="43.18" smashed="yes" rot="R90">
+<element name="C3" library="HyTechDevices" package="0805" value="47pF" x="55.372" y="43.18" smashed="yes" rot="R90">
 <attribute name="NAME" x="54.6481" y="43.18" size="0.3048" layer="25" rot="R90" align="bottom-center"/>
 <attribute name="VALUE" x="56.0832" y="43.18" size="0.3048" layer="27" rot="R90" align="top-center"/>
@@
 <attribute name="VALUE" x="52.578" y="40.386" size="0.6096" layer="28" rot="MR180" align="bottom-center"/>
 </element>
-<element name="C14" library="HyTechDevices" package="0805" value="5.3uF" x="52.07" y="49.022" smashed="yes">
+<element name="C14" library="HyTechDevices" package="0805" value="47pF" x="52.07" y="49.022" smashed="yes">
 <attribute name="NAME" x="52.07" y="49.7459" size="0.3048" layer="25" align="bottom-center"/>
 </element>
@@
 <attribute name="VALUE" x="52.324" y="47.752" size="0.6096" layer="28" rot="MR180" align="bottom-center"/>
 </element>
-<element name="C17" library="HyTechDevices" package="0805" value="5.3uF" x="54.864" y="55.88" smashed="yes" rot="MR180">
+<element name="C17" library="HyTechDevices" package="0805" value="47pF" x="54.864" y="55.88" smashed="yes" rot="MR180">
 <attribute name="NAME" x="54.864" y="55.1561" size="0.3048" layer="26" rot="MR180" align="bottom-center"/>
 <attribute name="VALUE" x="54.864" y="56.5912" size="0.3048" layer="28" rot="MR180" align="top-center"/>

Commit message: Main ECU rev2: Fixed capacitor values *again* (I can't math)
Parts:
- C14, C17, C3: value 47pF -> 47nF
Changed lines of the file:
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@@
 <attribute name="VALUE" x="64.008" y="40.386" size="0.6096" layer="28" rot="MR90" align="bottom-center"/>
 </element>
-<element name="C3" library="HyTechDevices" package="0805" value="47pF" x="55.372" y="43.18" smashed="yes" rot="R90">
+<element name="C3" library="HyTechDevices" package="0805" value="47nF" x="55.372" y="43.18" smashed="yes" rot="R90">
 <attribute name="NAME" x="54.6481" y="43.18" size="0.3048" layer="25" rot="R90" align="bottom-center"/>
 <attribute name="VALUE" x="56.0832" y="43.18" size="0.3048" layer="27" rot="R90" align="top-center"/>
@@
 <attribute name="VALUE" x="52.578" y="40.386" size="0.6096" layer="28" rot="MR180" align="bottom-center"/>
 </element>
-<element name="C14" library="HyTechDevices" package="0805" value="47pF" x="52.07" y="49.022" smashed="yes">
+<element name="C14" library="HyTechDevices" package="0805" value="47nF" x="52.07" y="49.022" smashed="yes">
 <attribute name="NAME" x="52.07" y="49.7459" size="0.3048" layer="25" align="bottom-center"/>
 </element>
@@
 <attribute name="VALUE" x="52.324" y="47.752" size="0.6096" layer="28" rot="MR180" align="bottom-center"/>
 </element>
-<element name="C17" library="HyTechDevices" package="0805" value="47pF" x="54.864" y="55.88" smashed="yes" rot="MR180">
+<element name="C17" library="HyTechDevices" package="0805" value="47nF" x="54.864" y="55.88" smashed="yes" rot="MR180">
 <attribute name="NAME" x="54.864" y="55.1561" size="0.3048" layer="26" rot="MR180" align="bottom-center"/>
 <attribute name="VALUE" x="54.864" y="56.5912" size="0.3048" layer="28" rot="MR180" align="top-center"/>

Commit message: Main ECU rev2/4: Add brake light NPN p/n
Parts:
- Q10: value (none) -> MMBT3904LT3G
Changed lines of the file:
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@@
 <attribute name="VALUE" x="59.6392" y="67.945" size="0.3048" layer="27" rot="R90" align="top-center"/>
 </element>
-<element name="Q10" library="HyTechDevices" package="SOT23" value="" x="59.182" y="49.022" smashed="yes" rot="MR0"/>
+<element name="Q10" library="HyTechDevices" package="SOT23" value="MMBT3904LT3G" x="59.182" y="49.022" smashed="yes" rot="MR0"/>
 <element name="U$15" library="HyTechDevices" package="SOT23" value="BJT_PNPSOT" x="58.928" y="54.61" smashed="yes" rot="MR90"/>
 <element name="R10" library="HyTechDevices" package="0805" value="2.2k" x="64.262" y="46.228" smashed="yes">

Commit message: Main ECU rev{2,4}: Specify PNP transistor P/Ns
Parts:
- U$15: value BJT_PNPSOT -> SMMBT2907ALT1G
Changed lines of the file:
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@@
 </element>
 <element name="Q10" library="HyTechDevices" package="SOT23" value="MMBT3904LT3G" x="59.182" y="49.022" smashed="yes" rot="MR0"/>
-<element name="U$15" library="HyTechDevices" package="SOT23" value="BJT_PNPSOT" x="58.928" y="54.61" smashed="yes" rot="MR90"/>
+<element name="U$15" library="HyTechDevices" package="SOT23" value="SMMBT2907ALT1G" x="58.928" y="54.61" smashed="yes" rot="MR90"/>
 <element name="R10" library="HyTechDevices" package="0805" value="2.2k" x="64.262" y="46.228" smashed="yes">
 <attribute name="NAME" x="64.262" y="46.9519" size="0.3048" layer="25" align="bottom-center"/>

Commit message: Main ECU rev{1-4}: Add warning about RTC cell assembly, specify current sensor input capacitor value, lower XBee LED resistor to 33R; Main ECU rev{2,4}: Specify MCP3208 input capacitor value; Main ECU rev4: Lower relay-controlling transistors' base resistor to 1k; Main ECU rev5: make all relevant changes previously listed
Parts:
- C10, C9: value (none) -> 0.1uF
- C11: value (none) -> 1uF
- R45: value 2.3k -> 33
Changed lines of the file:
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@@
 <attribute name="VALUE" x="56.4388" y="23.876" size="0.3048" layer="27" rot="R270" align="top-center"/>
 </element>
-<element name="C10" library="HyTechDevices" package="0805" value="" x="99.822" y="67.056" smashed="yes" rot="MR0">
+<element name="C10" library="HyTechDevices" package="0805" value="0.1uF" x="99.822" y="67.056" smashed="yes" rot="MR0">
 <attribute name="NAME" x="99.822" y="67.7799" size="0.3048" layer="26" rot="MR0" align="bottom-center" display="off"/>
 <attribute name="VALUE" x="99.822" y="66.3448" size="0.3048" layer="28" rot="MR0" align="top-center"/>
@@
 <attribute name="VALUE" x="88.3412" y="32.258" size="0.3048" layer="27" rot="R90" align="top-center"/>
 </element>
-<element name="C9" library="HyTechDevices" package="0805" value="" x="98.044" y="25.4" smashed="yes" rot="R180">
+<element name="C9" library="HyTechDevices" package="0805" value="0.1uF" x="98.044" y="25.4" smashed="yes" rot="R180">
 <attribute name="NAME" x="98.044" y="24.6761" size="0.3048" layer="25" rot="R180" align="bottom-center"/>
 <attribute name="VALUE" x="98.044" y="26.1112" size="0.3048" layer="27" rot="R180" align="top-center"/>
@@
 <attribute name="VALUE" x="79.5782" y="72.39" size="0.3048" layer="28" rot="MR270" align="top-center"/>
 </element>
-<element name="R45" library="HyTechDevices" package="0805" value="2.3k" x="24.638" y="33.782" smashed="yes" rot="R270">
+<element name="R45" library="HyTechDevices" package="0805" value="33" x="24.638" y="33.782" smashed="yes" rot="R270">
 <attribute name="NAME" x="25.3619" y="33.782" size="0.3048" layer="25" rot="R270" align="bottom-center"/>
 <attribute name="VALUE" x="23.9268" y="33.782" size="0.3048" layer="27" rot="R270" align="top-center"/>
@@
 <attribute name="VALUE" x="46.4058" y="32.385" size="0.3048" layer="27" rot="R270" align="top-center"/>
 </element>
-<element name="C11" library="HyTechDevices" package="0805" value="" x="46.99" y="35.814" smashed="yes">
+<element name="C11" library="HyTechDevices" package="0805" value="1uF" x="46.99" y="35.814" smashed="yes">
 <attribute name="NAME" x="46.99" y="36.5379" size="0.3048" layer="25" align="bottom-center"/>
 <attribute name="VALUE" x="46.99" y="35.1028" size="0.3048" layer="27" align="top-center"/>

Commit message: Main ECU rev{1-5}: Update values of LED resistors based on testing
Parts:
- R11: value 43 -> 150
- R14, R21: value 820 -> 2k
- R17: value 820 -> 20k
- R31: value 1.2K -> 6.8k
- R32: value 100 -> 1.2k
- R45: value 33 -> 0
Changed lines of the file:
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@@
 <attribute name="VALUE" x="94.5388" y="22.352" size="0.3048" layer="27" rot="R270" align="top-center"/>
 </element>
-<element name="R11" library="HyTechDevices" package="0805" value="43" x="29.21" y="69.342" smashed="yes" rot="MR180">
+<element name="R11" library="HyTechDevices" package="0805" value="150" x="29.21" y="69.342" smashed="yes" rot="MR180">
 <attribute name="NAME" x="29.21" y="68.6181" size="0.3048" layer="26" rot="MR180" align="bottom-center"/>
 <attribute name="VALUE" x="29.21" y="70.0532" size="0.3048" layer="28" rot="MR180" align="top-center"/>
@@
 <attribute name="VALUE" x="36.1188" y="68.326" size="0.3048" layer="28" rot="MR90" align="top-center"/>
 </element>
-<element name="R14" library="HyTechDevices" package="0805" value="820" x="30.734" y="55.118" smashed="yes" rot="MR180">
+<element name="R14" library="HyTechDevices" package="0805" value="2k" x="30.734" y="55.118" smashed="yes" rot="MR180">
 <attribute name="NAME" x="30.734" y="54.3941" size="0.3048" layer="26" rot="MR180" align="bottom-center"/>
 <attribute name="VALUE" x="30.734" y="55.8292" size="0.3048" layer="28" rot="MR180" align="top-center"/>
@@
 <attribute name="VALUE" x="20.7772" y="66.548" size="0.3048" layer="28" rot="MR270" align="top-center"/>
 </element>
-<element name="R17" library="HyTechDevices" package="0805" value="820" x="21.844" y="65.532" smashed="yes" rot="MR270">
+<element name="R17" library="HyTechDevices" package="0805" value="20k" x="21.844" y="65.532" smashed="yes" rot="MR270">
 <attribute name="NAME" x="21.1201" y="65.532" size="0.3048" layer="26" rot="MR270" align="bottom-center"/>
 <attribute name="VALUE" x="22.5552" y="65.532" size="0.3048" layer="28" rot="MR270" align="top-center"/>
@@
 <attribute name="VALUE" x="62.738" y="30.0228" size="0.3048" layer="27" align="top-center"/>
 </element>
-<element name="R21" library="HyTechDevices" package="0805" value="820" x="27.686" y="54.864" smashed="yes" rot="MR90">
+<element name="R21" library="HyTechDevices" package="0805" value="2k" x="27.686" y="54.864" smashed="yes" rot="MR90">
 <attribute name="NAME" x="28.4099" y="54.864" size="0.3048" layer="26" rot="MR90" align="bottom-center"/>
 <attribute name="VALUE" x="26.9748" y="54.864" size="0.3048" layer="28" rot="MR90" align="top-center"/>
@@
 <attribute name="VALUE" x="21.8948" y="33.782" size="0.3048" layer="27" rot="R270" align="top-center"/>
 </element>
-<element name="R31" library="HyTechDevices" package="0805" value="1.2K" x="13.462" y="57.404" smashed="yes" rot="MR180">
+<element name="R31" library="HyTechDevices" package="0805" value="6.8k" x="13.462" y="57.404" smashed="yes" rot="MR180">
 <attribute name="NAME" x="13.462" y="56.6801" size="0.3048" layer="26" rot="MR180" align="bottom-center" display="off"/>
 <attribute name="VALUE" x="13.462" y="58.1152" size="0.3048" layer="28" rot="MR180" align="top-center" display="off"/>
 </element>
-<element name="R32" library="HyTechDevices" package="0805" value="100" x="29.083" y="32.639" smashed="yes">
+<element name="R32" library="HyTechDevices" package="0805" value="1.2k" x="29.083" y="32.639" smashed="yes">
 <attribute name="NAME" x="29.083" y="33.3629" size="0.3048" layer="25" align="bottom-center"/>
 <attribute name="VALUE" x="29.083" y="31.9278" size="0.3048" layer="27" align="top-center"/>
@@
 <attribute name="VALUE" x="79.5782" y="72.39" size="0.3048" layer="28" rot="MR270" align="top-center"/>
 </element>
-<element name="R45" library="HyTechDevices" package="0805" value="33" x="24.638" y="33.782" smashed="yes" rot="R270">
+<element name="R45" library="HyTechDevices" package="0805" value="0" x="24.638" y="33.782" smashed="yes" rot="R270">
 <attribute name="NAME" x="25.3619" y="33.782" size="0.3048" layer="25" rot="R270" align="bottom-center"/>
 <attribute name="VALUE" x="23.9268" y="33.782" size="0.3048" layer="27" rot="R270" align="top-center"/>

Commit message: Main ECU rev{1-5}: Update values of OKI-78SR capacitors to 10uF
Parts:
- C1, C20: value .22uF -> 10uF
- C2, C21: value .1uF -> 10uF
Changed lines of the file:
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@@
 <attribute name="VALUE" x="91.948" y="38.1508" size="0.3048" layer="27" align="top-center"/>
 </element>
-<element name="C1" library="HyTechDevices" package="0805" value=".22uF" x="57.15" y="23.876" smashed="yes" rot="R270">
+<element name="C1" library="HyTechDevices" package="0805" value="10uF" x="57.15" y="23.876" smashed="yes" rot="R270">
 <attribute name="NAME" x="57.8739" y="23.876" size="0.3048" layer="25" rot="R270" align="bottom-center"/>
 <attribute name="VALUE" x="56.4388" y="23.876" size="0.3048" layer="27" rot="R270" align="top-center"/>
@@
 <attribute name="VALUE" x="99.822" y="66.3448" size="0.3048" layer="28" rot="MR0" align="top-center"/>
 </element>
-<element name="C2" library="HyTechDevices" package="0805" value=".1uF" x="59.69" y="29.21" smashed="yes" rot="R270">
+<element name="C2" library="HyTechDevices" package="0805" value="10uF" x="59.69" y="29.21" smashed="yes" rot="R270">
 <attribute name="NAME" x="60.4139" y="29.21" size="0.3048" layer="25" rot="R270" align="bottom-center"/>
 <attribute name="VALUE" x="58.9788" y="29.21" size="0.3048" layer="27" rot="R270" align="top-center"/>
@@
 <element name="U$16" library="HyTechDevices" package="CR-2450/G1AN" value="CR-2450/G1AN" x="78.994" y="10.668" smashed="yes" rot="R90"/>
 <element name="REG3" library="HyTechDevices" package="OKI-78SR" value="5V" x="53.34" y="33.528" smashed="yes" rot="MR0"/>
-<element name="C20" library="HyTechDevices" package="0805" value=".22uF" x="57.658" y="29.21" smashed="yes" rot="R270">
+<element name="C20" library="HyTechDevices" package="0805" value="10uF" x="57.658" y="29.21" smashed="yes" rot="R270">
 <attribute name="NAME" x="58.3819" y="29.21" size="0.3048" layer="25" rot="R270" align="bottom-center"/>
 <attribute name="VALUE" x="56.9468" y="29.21" size="0.3048" layer="27" rot="R270" align="top-center"/>
 </element>
-<element name="C21" library="HyTechDevices" package="0805" value=".1uF" x="47.117" y="32.385" smashed="yes" rot="R270">
+<element name="C21" library="HyTechDevices" package="0805" value="10uF" x="47.117" y="32.385" smashed="yes" rot="R270">
 <attribute name="NAME" x="47.8409" y="32.385" size="0.3048" layer="25" rot="R270" align="bottom-center"/>
 <attribute name="VALUE" x="46.4058" y="32.385" size="0.3048" layer="27" rot="R270" align="top-center"/>
