File: Board Designs/BMS/BMS Segment/BMS Segment rev9.sch (EAGLE design)
At the start: 113 parts

Commit message: BMS segment rev9: moved resistors, modified silkscreen
Parts:
- J: value (none) -> Jumper
- RB2_A, RB2_B: value 800R -> 806R
Changed lines of the file:
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@@
 <part name="C1_B" library="HyTechDevices" deviceset="CAP" device="0805" value="1uF"/>
 <part name="RB1_B" library="HyTechDevices" deviceset="RESISTOR" device="0805-RES" value="1K2"/>
-<part name="RB2_B" library="HyTechDevices" deviceset="RESISTOR" device="0805-RES" value="800R"/>
+<part name="RB2_B" library="HyTechDevices" deviceset="RESISTOR" device="0805-RES" value="806R"/>
 <part name="R1_B" library="HyTechDevices" deviceset="RESISTOR" device="0805-RES" value="100R"/>
 <part name="U$2" library="HyTechDevices" deviceset="LTC6804-2" device=""/>
@@
 <part name="C1_A" library="HyTechDevices" deviceset="CAP" device="0805" value="1uF"/>
 <part name="RB1_A" library="HyTechDevices" deviceset="RESISTOR" device="0805-RES" value="1K2"/>
-<part name="RB2_A" library="HyTechDevices" deviceset="RESISTOR" device="0805-RES" value="800R"/>
+<part name="RB2_A" library="HyTechDevices" deviceset="RESISTOR" device="0805-RES" value="806R"/>
 <part name="R1_A" library="HyTechDevices" deviceset="RESISTOR" device="0805-RES" value="100R"/>
 <part name="U$1" library="HyTechDevices" deviceset="LTC6804-2" device=""/>
@@
 <part name="SUPPLY57" library="supply1" deviceset="V-" device=""/>
 <part name="SUPPLY58" library="supply1" deviceset="V-" device=""/>
-<part name="J" library="HyTechDevices" deviceset="RESISTOR" device="0805-RES"/>
+<part name="J" library="HyTechDevices" deviceset="RESISTOR" device="0805-RES" value="Jumper"/>
 <part name="SUPPLY39" library="supply1" deviceset="V-" device=""/>
 <part name="SUPPLY59" library="supply2" deviceset="V-" device=""/>
@@
 <instance part="J" gate="G$1" x="-172.72" y="276.86" smashed="yes">
 <attribute name="NAME" x="-176.53" y="278.3586" size="1.778" layer="95"/>
-<attribute name="VALUE" x="-176.53" y="273.558" size="1.778" layer="96"/>
+<attribute name="VALUE" x="-173.99" y="273.558" size="1.778" layer="96"/>
 </instance>
 <instance part="SUPPLY39" gate="1" x="-101.6" y="134.62" smashed="yes">

Commit message: BMS rev9, HV rev10: Small adjustments for manufacturing
Parts:
- C6_A, C6_B, C7_A, C7_B: VOLTAGE (none) -> 100V
Changed lines of the file:
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@@
 <part name="U$2" library="HyTechDevices" deviceset="LTC6804-2" device=""/>
 <part name="C4_B" library="HyTechDevices" deviceset="CAP" device="0805" value="10nF"/>
-<part name="C6_B" library="HyTechDevices" deviceset="CAP" device="0805" value="0.1uF"/>
+<part name="C6_B" library="HyTechDevices" deviceset="CAP" device="0805" value="0.1uF">
+<attribute name="VOLTAGE" value="100V"/>
+</part>
 <part name="F9" library="HyTechDevices" deviceset="0001.2704.11" device="" value="0001.2704.11"/>
 <part name="F8" library="HyTechDevices" deviceset="0001.2704.11" device="" value="0001.2704.11"/>
@@
 <part name="U$1" library="HyTechDevices" deviceset="LTC6804-2" device=""/>
 <part name="C4_A" library="HyTechDevices" deviceset="CAP" device="0805" value="10nF"/>
-<part name="C6_A" library="HyTechDevices" deviceset="CAP" device="0805" value="0.1uF"/>
+<part name="C6_A" library="HyTechDevices" deviceset="CAP" device="0805" value="0.1uF">
+<attribute name="VOLTAGE" value="100V"/>
+</part>
 <part name="F18" library="HyTechDevices" deviceset="0001.2704.11" device="" value="0001.2704.11"/>
 <part name="F17" library="HyTechDevices" deviceset="0001.2704.11" device="" value="0001.2704.11"/>
@@
 <part name="THERM3_B" library="HyTechDevices" deviceset="CONNECTOR-2" device="NANO-FIT_VERTICAL-2" value="Th1"/>
 <part name="U$3" library="HyTechDevices" deviceset="NSV1C201MZ4" device=""/>
-<part name="C7_A" library="HyTechDevices" deviceset="CAP" device="0805" value="0.1uF"/>
+<part name="C7_A" library="HyTechDevices" deviceset="CAP" device="0805" value="0.1uF">
+<attribute name="VOLTAGE" value="100V"/>
+</part>
 <part name="SUPPLY69" library="supply1" deviceset="V-" device=""/>
 <part name="RIN_A" library="HyTechDevices" deviceset="RESISTOR" device="0805-RES" value="100R"/>
@@
 <part name="SUPPLY40" library="supply1" deviceset="V-" device=""/>
 <part name="U$4" library="HyTechDevices" deviceset="NSV1C201MZ4" device=""/>
-<part name="C7_B" library="HyTechDevices" deviceset="CAP" device="0805" value="0.1uF"/>
+<part name="C7_B" library="HyTechDevices" deviceset="CAP" device="0805" value="0.1uF">
+<attribute name="VOLTAGE" value="100V"/>
+</part>
 <part name="RIN_B" library="HyTechDevices" deviceset="RESISTOR" device="0805-RES" value="100R"/>
 <part name="C8_B" library="HyTechDevices" deviceset="CAP" device="0805" value="1uF"/>
@@
 <attribute name="NAME" x="-110.744" y="98.679" size="1.778" layer="95" rot="R180"/>
 <attribute name="VALUE" x="-110.744" y="103.759" size="1.778" layer="96" rot="R180"/>
+<attribute name="VOLTAGE" x="-110.744" y="106.68" size="1.778" layer="96" rot="R180"/>
 </instance>
 <instance part="F9" gate="G$1" x="-210.82" y="137.16" smashed="yes">
@@
 <attribute name="NAME" x="-110.744" y="337.439" size="1.778" layer="95" rot="R180"/>
 <attribute name="VALUE" x="-110.744" y="342.519" size="1.778" layer="96" rot="R180"/>
+<attribute name="VOLTAGE" x="-110.744" y="345.44" size="1.778" layer="96" rot="R180"/>
 </instance>
 <instance part="F18" gate="G$1" x="-210.82" y="279.4" smashed="yes">
@@
 <attribute name="NAME" x="-98.044" y="350.901" size="1.778" layer="95" rot="MR0"/>
 <attribute name="VALUE" x="-98.044" y="345.821" size="1.778" layer="96" rot="MR0"/>
+<attribute name="VOLTAGE" x="-98.044" y="342.9" size="1.778" layer="96" rot="MR0"/>
 </instance>
 <instance part="SUPPLY69" gate="1" x="-96.52" y="340.36" smashed="yes">
@@
 <attribute name="NAME" x="-98.044" y="112.141" size="1.778" layer="95" rot="MR0"/>
 <attribute name="VALUE" x="-98.044" y="107.061" size="1.778" layer="96" rot="MR0"/>
+<attribute name="VOLTAGE" x="-98.044" y="104.14" size="1.778" layer="96" rot="MR0"/>
 </instance>
 <instance part="RIN_B" gate="G$1" x="-121.92" y="114.3" smashed="yes">

Commit message: BMS rev9: Added termination resistor silkscreen
Parts:
- RM_A, RM_B: TYPE (none) -> TERMINATION
Changed lines of the file:
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@@
 <setting verticaltext="up"/>
 </settings>
-<grid distance="0.1" unitdist="inch" unit="inch" style="lines" multiple="1" display="no" altdistance="0.01" altunitdist="inch" altunit="inch"/>
+<grid distance="1" unitdist="mm" unit="mm" style="lines" multiple="1" display="no" altdistance="0.01" altunitdist="inch" altunit="mm"/>
 <layers>
 <layer number="1" name="Top" color="4" fill="1" visible="no" active="no"/>
@@
 <part name="RU1_B" library="HyTechDevices" deviceset="RESISTOR" device="0805-RES" value="100R"/>
 <part name="TRANSFORMER" library="HyTechDevices" deviceset="HM2102NLT" device="" value="HM2102NLT"/>
-<part name="RM_B" library="HyTechDevices" deviceset="RESISTOR" device="0805-RES" value="100R"/>
+<part name="RM_B" library="HyTechDevices" deviceset="RESISTOR" device="0805-RES" value="100R">
+<attribute name="TYPE" value="TERMINATION"/>
+</part>
 <part name="R4_B" library="HyTechDevices" deviceset="RESISTOR" device="0805-RES" value="22R"/>
 <part name="R5_B" library="HyTechDevices" deviceset="RESISTOR" device="0805-RES" value="22R"/>
@@
 <part name="C5_A" library="HyTechDevices" deviceset="CAP" device="0805" value="10nF"/>
 <part name="RU1_A" library="HyTechDevices" deviceset="RESISTOR" device="0805-RES" value="100R"/>
-<part name="RM_A" library="HyTechDevices" deviceset="RESISTOR" device="0805-RES" value="100R"/>
+<part name="RM_A" library="HyTechDevices" deviceset="RESISTOR" device="0805-RES" value="100R">
+<attribute name="TYPE" value="TERMINATION"/>
+</part>
 <part name="R4_A" library="HyTechDevices" deviceset="RESISTOR" device="0805-RES" value="22R"/>
 <part name="R5_A" library="HyTechDevices" deviceset="RESISTOR" device="0805-RES" value="22R"/>
@@
 </instance>
 <instance part="RM_B" gate="G$1" x="40.64" y="111.76" smashed="yes" rot="R270">
-<attribute name="NAME" x="42.1386" y="115.57" size="1.778" layer="95" rot="R270"/>
+<attribute name="NAME" x="45.1386" y="115.57" size="1.778" layer="95" rot="R270"/>
 <attribute name="VALUE" x="37.338" y="115.57" size="1.778" layer="96" rot="R270"/>
+<attribute name="TYPE" x="42.64" y="119.76" size="1.778" layer="96" rot="R270"/>
 </instance>
 <instance part="R4_B" gate="G$1" x="33.02" y="121.92" smashed="yes">
@@
 </instance>
 <instance part="RM_A" gate="G$1" x="40.64" y="350.52" smashed="yes" rot="R270">
-<attribute name="NAME" x="42.1386" y="354.33" size="1.778" layer="95" rot="R270"/>
+<attribute name="NAME" x="44.6786" y="354.33" size="1.778" layer="95" rot="R270"/>
 <attribute name="VALUE" x="37.338" y="354.33" size="1.778" layer="96" rot="R270"/>
+<attribute name="TYPE" x="42.18" y="358.14" size="1.778" layer="96" rot="R270"/>
 </instance>
 <instance part="R4_A" gate="G$1" x="33.02" y="360.68" smashed="yes">
