File: Board Designs/External Boards/Charger Relay Board/ChargerRelayBoardRev1.brd (EAGLE design)
At the start: 46.3 x 34.1 mm, 4 parts, among them X1 CONNECTOR-2, X2 CONNECTOR-2

Commit message: Modified charger board silkscreens for manufacturing
Other:
- board text added: "CONTROL"
- board text added: "SWITCHED"
Changed lines of the file:
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@@
 <?xml version="1.0" encoding="utf-8"?>
 <!DOCTYPE eagle SYSTEM "eagle.dtd">
-<eagle version="9.1.3">
+<eagle version="9.2.2">
 <drawing>
 <settings>
@@
 <hole x="61" y="35" drill="3.175"/>
 <text x="58" y="6" size="1.016" layer="51" font="vector" rot="R180">HyTech Racing 2019 Charger Relay Board Rev1</text>
+<text x="26" y="22" size="1.524" layer="51" font="vector" rot="R270" align="bottom-center">CONTROL</text>
+<text x="55" y="22" size="1.524" layer="51" font="vector" rot="R90" align="bottom-center">SWITCHED</text>
 </plain>
 <attributes>
@@
 </autorouter>
 <elements>
-<element name="D2" library="HyTechDevices" package="0805_D" value="DIODE0805" x="29.13" y="21.59" rot="R270"/>
-<element name="X1" library="HyTechDevices" package="MINIFIT_5566-2" value="CONNECTOR-2" x="58.5" y="21.87">
+<element name="D2" library="HyTechDevices" package="0805_D" value="DIODE0805" x="29.13" y="21.59" smashed="yes" rot="R270">
+<attribute name="NAME" x="29.8539" y="21.59" size="0.3048" layer="25" rot="R270" align="bottom-center"/>
+<attribute name="VALUE" x="28.4188" y="21.59" size="0.3048" layer="27" rot="R270" align="top-center"/>
+</element>
+<element name="X1" library="HyTechDevices" package="MINIFIT_5566-2" value="CONNECTOR-2" x="58.5" y="21.87" smashed="yes">
 <attribute name="MF" value="" x="58.5" y="21.87" size="1.778" layer="27" display="off"/>
 <attribute name="MPN" value="" x="58.5" y="21.87" size="1.778" layer="27" display="off"/>
+<attribute name="NAME" x="58.5" y="16.663" size="0.8128" layer="25" rot="R180" align="bottom-center"/>
 <attribute name="OC_FARNELL" value="1822072" x="58.5" y="21.87" size="1.778" layer="27" display="off"/>
 <attribute name="OC_NEWARK" value="unknown" x="58.5" y="21.87" size="1.778" layer="27" display="off"/>
+<attribute name="VALUE" x="58.5" y="28.728" size="0.8128" layer="27" align="bottom-center"/>
 </element>
-<element name="X2" library="HyTechDevices" package="MINIFIT_5566-2" value="CONNECTOR-2" x="22.32" y="21.59">
+<element name="X2" library="HyTechDevices" package="MINIFIT_5566-2" value="CONNECTOR-2" x="22.32" y="21.59" smashed="yes">
 <attribute name="MF" value="" x="22.32" y="21.59" size="1.778" layer="27" display="off"/>
 <attribute name="MPN" value="" x="22.32" y="21.59" size="1.778" layer="27" display="off"/>
+<attribute name="NAME" x="22.32" y="16.383" size="0.8128" layer="25" rot="R180" align="bottom-center"/>
 <attribute name="OC_FARNELL" value="1822072" x="22.32" y="21.59" size="1.778" layer="27" display="off"/>
 <attribute name="OC_NEWARK" value="unknown" x="22.32" y="21.59" size="1.778" layer="27" display="off"/>
+<attribute name="VALUE" x="22.32" y="28.448" size="0.8128" layer="27" align="bottom-center"/>
 </element>
-<element name="U$1" library="HyTechDevices" package="KT12-1A-40L-THT" value="KT12-1A-40L-THT" x="46.99" y="6.35" rot="R90"/>
+<element name="U$1" library="HyTechDevices" package="KT12-1A-40L-THT" value="KT12-1A-40L-THT" x="46.99" y="6.35" smashed="yes" rot="R90"/>
 </elements>
 <signals>
