File: External Diagram FH0.sch (EAGLE design)
At the start: 74 parts

Commit message: New wiring harness diagram with Main ECU in front of firewall
Parts:
- removed BUTTON_MC_CYCLE: SWITCH_SPST_MOM, HyTechSymbols:SWITCH_SPST_MOM
- removed FIREWALL_3: 8STA01204PN, HyTechSymbols:M04
- removed FIREWALL_4: 8STA61204SN, HyTechSymbols:M04
- removed LED_MC_ERR: LED, HyTechSymbols:LED
- added BUTTON_CYCLE: SWITCH_SPST_MOM, HyTechSymbols:SWITCH_SPST_MOM
- added LED_POWER: LED, HyTechSymbols:LED
- FIREWALL_1: value 8STA01035PN -> 8STA01435PN; device HyTechSymbols:M13 -> HyTechSymbols:M37
- FIREWALL_2: value 8STA61035SN -> 8STA61435SN; device HyTechSymbols:M13 -> HyTechSymbols:M37
Connections:
- removed net 12V_ACCUM_MAINT: FIREWALL_2.4, MAIN_PRIM_2.10
- removed net 12V_DASH: MAIN_PRIM_1.34
- removed net 12V_MAINT: MAINTENANCE.7
- removed net CANH_FRONT: FIREWALL_2.6, MAIN_PRIM_2.12
- removed net CANL_FRONT: FIREWALL_2.5, MAIN_PRIM_2.11
- removed net GND_ACCUM_RELAYS: ACCUM_2.13
- removed net GND_DASH: BUTTON_MARK.S, BUTTON_MC_CYCLE.S, BUTTON_MODE.S, BUTTON_START.S, DASH_1.1, DASH_2.1, LED_BMS.C, LED_IMD.C, LED_MC_ERR.C, LED_MODE.C, LED_START.C, MAIN_PRIM_2.36, RTDS.2
- removed net GND_MAIN_ECU: FIREWALL_3.4, FIREWALL_4.4, MAIN_SEC_2.4
- removed net GND_MC: U$1.GND, U$1.J2-6/GND
- removed net GND_MEASURE: MEASURE_GND.1
- removed net GND_SHIELD: FIREWALL_1.1, FIREWALL_2.1
- removed net MOTOR_SHIELD: U$1.J2-19/SHIELD_GND
- new net 12V_DASH/MAINT: DASH_1.1, FIREWALL_1.1, FIREWALL_2.1, MAINTENANCE.7, MAIN_PRIM_1.34, MAIN_PRIM_2.34
- net 12VSUPPLY_BRB: no longer FIREWALL_3.1, FIREWALL_4.1
- net 12V_ACCUM: now also MAIN_PRIM_2.10; no longer FIREWALL_1.4
- net 5V_ACCEL_1: now also FIREWALL_1.14, FIREWALL_2.14
- net 5V_ACCEL_2: now also FIREWALL_1.17, FIREWALL_2.17
- net 5V_BRAKE: now also FIREWALL_1.20, FIREWALL_2.20
- net BMS_OK: no longer FIREWALL_1.9, FIREWALL_2.9
- net BRAKE_LIGHT: no longer FIREWALL_1.3, FIREWALL_2.3
- net CANH_ACCUM: now also MAIN_PRIM_2.13
- net CANH_MC: now also MAIN_PRIM_2.12; no longer FIREWALL_1.6
- net CANL_ACCUM: now also MAIN_PRIM_2.26; no longer FIREWALL_1.5
- net CANL_MC: now also MAIN_PRIM_2.11
- net DASH_1: now also FIREWALL_1.2, FIREWALL_2.2
- net DASH_10: now also FIREWALL_1.11, FIREWALL_2.11
- net DASH_11: now also FIREWALL_1.12, FIREWALL_2.12
- net DASH_12: now also FIREWALL_1.13, FIREWALL_2.13
- net DASH_2: now also FIREWALL_1.3, FIREWALL_2.3
- net DASH_3: now also FIREWALL_1.4, FIREWALL_2.4
- net DASH_4: now also FIREWALL_1.5, FIREWALL_2.5
- net DASH_5: now also FIREWALL_1.6, FIREWALL_2.6, LED_POWER.A; no longer LED_MC_ERR.A
- net DASH_6: now also FIREWALL_1.7, FIREWALL_2.7
- net DASH_7: now also FIREWALL_1.8, FIREWALL_2.8
- net DASH_8: now also FIREWALL_1.9, FIREWALL_2.9
- net DASH_9: now also BUTTON_CYCLE.P, FIREWALL_1.10, FIREWALL_2.10; no longer BUTTON_MC_CYCLE.P
- net GND: now also ACCUM_2.13, BUTTON_CYCLE.S, BUTTON_MARK.S, BUTTON_MODE.S, BUTTON_START.S, LED_BMS.C, LED_IMD.C, LED_MODE.C, LED_POWER.C, LED_START.C, MAIN_SEC_2.4, MEASURE_GND.1, RTDS.2, U$1.J2-6/GND
- net GND_ACCEL_1: now also FIREWALL_1.15, FIREWALL_2.15
- net GND_ACCEL_2: now also FIREWALL_1.18, FIREWALL_2.18
- net GND_ACCUM: no longer FIREWALL_2.8
- net GND_BRAKE: now also FIREWALL_1.21, FIREWALL_2.21
- net GND_MAINT: now also MAIN_PRIM_2.36; no longer FIREWALL_1.8
- net IMD_OKHS: no longer FIREWALL_1.10, FIREWALL_2.10
- net INVERTER_SUPPLY: no longer FIREWALL_1.2, FIREWALL_2.2
- net LATCH_EXT_BTN: no longer FIREWALL_1.11, FIREWALL_2.11
- net RET_FAN_1: no longer FIREWALL_1.7, FIREWALL_2.7
- net RET_FAN_2: no longer FIREWALL_3.3, FIREWALL_4.3
- net RET_PUMP_1: no longer FIREWALL_3.2, FIREWALL_4.2
- net SHUTDOWN_D: now also FIREWALL_1.23, FIREWALL_2.23
- net SHUTDOWN_F: now also FIREWALL_1.24, FIREWALL_2.24; no longer FIREWALL_1.12, FIREWALL_2.12
- net SIGNAL_ACCEL_1: now also FIREWALL_1.16, FIREWALL_2.16
- net SIGNAL_ACCEL_2: now also FIREWALL_1.19, FIREWALL_2.19
- net SIGNAL_BRAKE: now also FIREWALL_1.22, FIREWALL_2.22
- net SSOK: now also FIREWALL_1.25, FIREWALL_2.25; no longer FIREWALL_1.13, FIREWALL_2.13
Other:
- note added: "12AWG grounding per FH EV4.1.4"
- note added: "TODO Rectify diff w Parker"
- note removed: "12AWG chassis grounding per FH EV4.1.4"
- moved on the sheet: ACCUM_1, ACCUM_2, AIR1, AIR2, AMS_TEST_1, AMS_TEST_2, BMS_IMD_LATCH_BTN, BOTS, BRAKE_LIGHT, BUTTON_MARK, BUTTON_MODE, BUTTON_START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
