File: External Diagram FH1.sch (EAGLE design)
At the start: 72 parts

Commit message: New wiring harness diagram with Main ECU in front of firewall
Parts:
- added ACCUMULATOR_FAN_1, ACCUMULATOR_FAN_2, BRL_1, BRL_2, PUMP_1, PUMP_2, RADIATOR_FAN_1, RADIATOR_FAN_2, TSAL1, TSAL2: ASMPP30-1X2-RK, HyTechSymbols:M02
- added BRAKE_1: 8STA00235PN, HyTechSymbols:M03
- added BRAKE_2: 8STA60235SN, HyTechSymbols:M03
- added FIREWALL_3: 8STA01204PN, HyTechSymbols:M04
- added FIREWALL_4: 8STA61204SN, HyTechSymbols:M04
- added LED_SSOK: YELLOW, HyTechSymbols:LED
- added PED_1: 8STA01035PN, HyTechSymbols:M13
- added PED_2: 8STA61035SN, HyTechSymbols:M13
- DASH_1: value 8STA61035SN -> 8STA01035PN
- DASH_2: value 8STA01035PN -> 8STA61035SN
- FIREWALL_1: value 8STA01435PN -> 8STA01035PN; device HyTechSymbols:M37 -> HyTechSymbols:M13
- FIREWALL_2: value 8STA01435PN -> 8STA61035SN; device HyTechSymbols:M37 -> HyTechSymbols:M13
- LED_BMS, LED_IMD, LED_MC_ERR: value LED -> RED
- LED_MODE: value LED -> GREEN
- LED_START: value LED -> BLUE
- MOTOR_RESOLVER_1: value 8STA00835PN -> 8STA60835SN
- MOTOR_RESOLVER_2: value 8STA60835SN -> 8STA00835PN
- MOTOR_TEMP_1: value 8STA00235PN -> 8STA60235SN
- MOTOR_TEMP_2: value 8STA60235SN -> 8STA00235PN
Connections:
- removed net 12VSUPPLY_COOLING: S1.O
- removed net GND_MEASURE: MEASURE_GND.1
- new net 12VSUPPLY_COOLING_FAN_1: ACCUMULATOR_FAN_1.1, ACCUMULATOR_FAN_2.1
- new net 12VSUPPLY_COOLING_FAN_2: RADIATOR_FAN_1.1, RADIATOR_FAN_2.1
- new net 12VSUPPLY_COOLING_PUMP_1: PUMP_1.1, PUMP_2.1, S1.O
- new net 12V_ACCUM_MAINT: FIREWALL_2.4, MAIN_PRIM_2.10
- new net GND_BR: BRAKE_LIGHT.C, BRL_1.1, BRL_2.1
- new net GND_LEFT_PANEL_BR: LEFT_SSOK.C
- new net GND_RIGHT_PANEL: BMS_IMD_LATCH_BTN.S, MEASURE_GND.1, RIGHT_SSOK.C, TSAL1.2
- new net N$3: TSAL.A, TSAL2.1
- new net N$4: TSAL.C, TSAL2.2
- new net SHUTDOWN_E: BOTS.O, COCKPIT_BRB.P, DASH_2.12, LED_SSOK.A, PED_1.13, PED_2.13
- net 12VSUPPLY_BRB: now also FIREWALL_3.1, FIREWALL_4.1
- net 12V_ACCUM: now also FIREWALL_1.4; no longer MAIN_PRIM_2.10
- net 12V_DASH: no longer FIREWALL_1.17, FIREWALL_2.17, MAIN_PRIM_2.34
- net 5V_ACCEL_1: now also PED_1.6, PED_2.6; no longer FIREWALL_1.19, FIREWALL_2.19
- net 5V_ACCEL_2: now also PED_1.2, PED_2.2; no longer FIREWALL_1.22, FIREWALL_2.22
- net 5V_BRAKE: now also BRAKE_1.1, BRAKE_2.1; no longer FIREWALL_1.26, FIREWALL_2.26
- net BMS_OK: now also FIREWALL_1.9, FIREWALL_2.9
- net BRAKE_LIGHT: now also BRL_1.2, BRL_2.2, FIREWALL_1.3, FIREWALL_2.3
- net CANH_ACCUM: no longer MAIN_PRIM_2.13
- net CANH_FRONT: now also FIREWALL_2.6, MAIN_PRIM_2.12; no longer FIREWALL_1.34
- net CANH_MC: now also FIREWALL_1.6; no longer MAIN_PRIM_2.12
- net CANL_ACCUM: now also FIREWALL_1.5; no longer MAIN_PRIM_2.26
- net CANL_FRONT: now also FIREWALL_2.5, MAIN_PRIM_2.11; no longer FIREWALL_1.33
- net CANL_MC: no longer MAIN_PRIM_2.11
- net DASH_1: no longer FIREWALL_1.3, FIREWALL_2.3
- net DASH_10: no longer FIREWALL_1.13, FIREWALL_2.13
- net DASH_11: no longer FIREWALL_1.14, FIREWALL_2.14
- net DASH_12: no longer FIREWALL_1.16, FIREWALL_2.16
- net DASH_2: no longer FIREWALL_1.4, FIREWALL_2.4
- net DASH_3: no longer FIREWALL_1.5, FIREWALL_2.5
- net DASH_4: no longer FIREWALL_1.6, FIREWALL_2.6
- net DASH_5: no longer FIREWALL_1.7, FIREWALL_2.7
- net DASH_6: no longer FIREWALL_1.9, FIREWALL_2.9
- net DASH_7: no longer FIREWALL_1.10, FIREWALL_2.10
- net DASH_8: no longer FIREWALL_1.11, FIREWALL_2.11
- net DASH_9: no longer FIREWALL_1.12, FIREWALL_2.12
- net GND: no longer BMS_IMD_LATCH_BTN.S, BRAKE_LIGHT.C, LEFT_SSOK.C, RIGHT_SSOK.C, TSAL.C
- net GND_ACCEL_1: now also PED_1.5, PED_2.5; no longer FIREWALL_1.20, FIREWALL_2.20
- net GND_ACCEL_2: now also PED_1.1, PED_2.1; no longer FIREWALL_1.23, FIREWALL_2.23
- net GND_ACCUM: now also FIREWALL_2.8
- net GND_BRAKE: now also BRAKE_1.2, BRAKE_2.2; no longer FIREWALL_1.27, FIREWALL_2.27
- net GND_DASH: now also LED_SSOK.C; no longer FIREWALL_1.2, FIREWALL_2.2
- net GND_MAINT: now also FIREWALL_1.8
- net GND_MAIN_ECU: now also FIREWALL_3.4, FIREWALL_4.4
- net GND_SHIELD: no longer FIREWALL_1.15, FIREWALL_1.18, FIREWALL_1.25, FIREWALL_1.32, FIREWALL_1.8, FIREWALL_2.15, FIREWALL_2.18, FIREWALL_2.25, FIREWALL_2.8
- net IMD_OKHS: now also FIREWALL_1.10, FIREWALL_2.10
- net INVERTER_SUPPLY: now also FIREWALL_1.2, FIREWALL_2.2
- net LATCH_EXT_BTN: now also FIREWALL_1.11, FIREWALL_2.11
- net RET_FAN_1: now also ACCUMULATOR_FAN_1.2, ACCUMULATOR_FAN_2.2, FIREWALL_1.7, FIREWALL_2.7
- net RET_FAN_2: now also FIREWALL_3.3, FIREWALL_4.3, RADIATOR_FAN_1.2, RADIATOR_FAN_2.2
- net RET_PUMP_1: now also FIREWALL_3.2, FIREWALL_4.2, PUMP_1.2, PUMP_2.2
- net SHUTDOWN_D: now also PED_1.12, PED_2.12; no longer FIREWALL_1.29, FIREWALL_2.29
- net SHUTDOWN_F: now also FIREWALL_1.12, FIREWALL_2.12; no longer FIREWALL_1.30, FIREWALL_2.30
- net SIGNAL_ACCEL_1: now also PED_1.3, PED_2.3; no longer FIREWALL_1.21, FIREWALL_2.21
- net SIGNAL_ACCEL_2: now also PED_1.4, PED_2.4; no longer FIREWALL_1.24, FIREWALL_2.24
- net SIGNAL_BRAKE: now also BRAKE_1.3, BRAKE_2.3; no longer FIREWALL_1.28, FIREWALL_2.28
- net SSOK: now also FIREWALL_1.13, FIREWALL_2.13; no longer BOTS.O, COCKPIT_BRB.P, DASH_2.12, FIREWALL_1.31, FIREWALL_2.31
- net TSAL: now also TSAL1.1; no longer TSAL.A
Other:
- note added: "Firewall"
- note added: "Pedal Box"
- moved on the sheet: ACCUM_1, ACCUM_2, AIR1, AIR2, AMS_TEST_1, AMS_TEST_2, BMS_IMD_LATCH_BTN, BOTS, BRAKE_LIGHT, BUTTON_MARK, BUTTON_MC_CYCLE, BUTTON_MODE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
